File: subharmolizer-rev2/subharmolizer-schem.kicad_sch (KiCad schematic)
At the start: 60 parts, among them J1 Audio IN, J2 Audio OUT, J3 Subharm CV IN, Q1 2N3904, U1 TL072, U2 74HC00, U3 CD4516B, U4 LM311, U5 74LS74

Commit message: rev2 tweaks
Parts:
- added C12: 4n7, symbol Device:C
- added RV2: 100k Log, symbol Device:R_Potentiometer
- added TP6: Sqr_Input, symbol Connector:TestPoint
- R5: value 10k -> 22k
Connections:
- net GND: now also C12.1, RV2.3
- net at C1.2: now also RV2.1; no longer R1.1
- net at D1.1 (K), R5.2, R6.1: now also TP6.1
- net at D4.2 (A), D5.1 (K), R1.2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: now also C12.2
- new net: R1.1, RV2.2
Other:
- moved on the sheet: C1, C2, C3, C9, D1, D4, D5, J1, R1, R2, R24, R3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
